File: esp32/kicad/ESP32-li-ion-cell-monitor/ESP32-li-ion-cell-monitor.sch (KiCad schematic (older format))
At the start: 43 parts, among them J1 Conn_01x01_Female, J2 Conn_01x01_Female, J3 Conn_01x05_Male, Q1 Q_NMOS_GSD, Q2 Q_NMOS_GSD, Q3 Q_NMOS_GSD, Q4 Q_NMOS_GSD, U1 NCP186B, U2 ESP-WROOM-32, U3 INA219_SOT23-8, U4 Si7060-00, U5 Si7060-01

Commit message: ESP32-li-ion-cell-monitor
Parts:
- U2: symbol module:ES-WROOM-32 -> module:ESP-WROOM-32
Changed lines of the file:
@@
 $EndDescr
 $Comp
-L module:ES-WROOM-32 U2
+L module:ESP-WROOM-32 U2
 U 1 1 5B3380F2
 P 2700 5200
